File: pcb/qnode8.sch (EAGLE design)
At the start: 65 parts, among them IC1 STM32F401CCU6, IC2 S25FL064K, IC3 LM3671MF-ADJ, IC4 AX5243, IC5 MCP73831-2ATI/OT, X1 BU-SMA-G, X2 USB-MICROB

Commit message: Finish schematic and board layout
Parts:
- removed LED2: (no value), led:LED3MM
- removed SWGND: WIREPADSMD5-1,8, wirepad:WIREPADSMD5-1,8
- removed U$1, U$2: XTAL-7M, qyx-misc:XTAL-7M
- added ANT: BU-SMA-G, con-coax:BU-SMA-G
- added C20: 10nF, rcl:C-EUC0603
- added GND: TPB2,54, testpad:TPB2,54
- added L2: FB, rcl:L-USL2012C
- added R8: 470R, rcl:R-EU_R0603
- added ST: (no value), led:LED3MM
- added USB: USB-MICROB, SparkFun:USB-MICROB
- BAT: value (none) -> 332-02; device SparkFun:M02POLAR -> con-garry:332-02
- RX, SWCLK, SWDIO, TX, VBAT: value WIREPADSMD5-1,8 -> TPB2,54; device wirepad:WIREPADSMD5-1,8 -> testpad:TPB2,54
- X1: value BU-SMA-G -> XTAL-7M; device con-coax:BU-SMA-G -> qyx-misc:XTAL-7M
- X2: value USB-MICROB -> XTAL-7M; device SparkFun:USB-MICROB -> qyx-misc:XTAL-7M
Connections:
- removed net LED_STAT: IC1.PA3
- new net BTN1: IC1.PA0, S1.S
- new net LED1: IC1.PA1, R8.2
- new net N$23: R8.1, ST.C
- new net N$24: C20.1, L2.1, USB.VBUS
- net +3V3: now also S1.P, ST.A
- net CHG_STAT: now also IC1.PB2
- net CON_RX: now also RX.TP; no longer RX.P
- net CON_TX: now also TX.TP; no longer TX.P
- net GND: now also ANT.2, BAT-2.S, C20.2, GND.TP, USB.GND, X1.G1, X1.G2, X2.G1, X2.G2; no longer BAT.1, SWGND.P, U$1.G1, U$1.G2, U$2.G1, U$2.G2, X1.2, X2.GND
- net N$14: now also ANT.1; no longer X1.1
- net N$20: now also X2.2; no longer U$2.2
- net N$21: now also X2.1; no longer U$2.1
- net N$8: now also X1.1; no longer U$1.1
- net N$9: now also X1.2; no longer U$1.2
- net SWCLK: now also SWCLK.TP; no longer SWCLK.P
- net SWDIO: now also SWDIO.TP; no longer SWDIO.P
- net USB_DM: now also USB.D-; no longer X2.D-
- net USB_DP: now also USB.D+; no longer X2.D+
- net VBAT: now also BAT-1.S, VBAT.TP; no longer BAT.2, VBAT.P
- net VUSB: now also L2.2; no longer X2.VBUS
Other:
- note added: "(c) qyx@krtko.org, CC-BY-SA"
- note added: "qNode8-1.0.0+20160811"
- note removed: "(1 cell 4.2V, charging current ~450mA)"
- note removed: "qNode4, (c) qyx@krtko.org, rev1 (20140703), CC-BY-SA"
- moved on the sheet: C1, C10, C11, C12, C13, C14, C15, C16, C17, C18, C19, C2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

Commit message: Fix unconnected USB_VBUS
Connections:
- net N$24 renamed USB_VBUS
- net VUSB: now also IC1.PA9
Other:
- note added: "qNode8-1.0.1+20160812"
- note removed: "qNode8-1.0.0+20160811"
- moved on the sheet: C20
Changed lines of the file:
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@@
 <grid distance="0.1" unitdist="inch" unit="inch" style="lines" multiple="1" display="no" altdistance="0.01" altunitdist="inch" altunit="inch"/>
 <layers>
-<layer number="1" name="Top" color="4" fill="1" visible="yes" active="no"/>
-<layer number="16" name="Bottom" color="1" fill="1" visible="yes" active="no"/>
-<layer number="17" name="Pads" color="2" fill="1" visible="yes" active="no"/>
-<layer number="18" name="Vias" color="2" fill="1" visible="yes" active="no"/>
-<layer number="19" name="Unrouted" color="6" fill="1" visible="yes" active="no"/>
-<layer number="20" name="Dimension" color="15" fill="1" visible="yes" active="no"/>
-<layer number="21" name="tPlace" color="7" fill="1" visible="yes" active="no"/>
-<layer number="22" name="bPlace" color="7" fill="1" visible="yes" active="no"/>
-<layer number="23" name="tOrigins" color="15" fill="1" visible="yes" active="no"/>
-<layer number="24" name="bOrigins" color="15" fill="1" visible="yes" active="no"/>
-<layer number="25" name="tNames" color="7" fill="1" visible="yes" active="no"/>
-<layer number="26" name="bNames" color="7" fill="1" visible="yes" active="no"/>
-<layer number="27" name="tValues" color="7" fill="1" visible="yes" active="no"/>
-<layer number="28" name="bValues" color="7" fill="1" visible="yes" active="no"/>
+<layer number="1" name="Top" color="4" fill="1" visible="no" active="no"/>
+<layer number="16" name="Bottom" color="1" fill="1" visible="no" active="no"/>
+<layer number="17" name="Pads" color="2" fill="1" visible="no" active="no"/>
+<layer number="18" name="Vias" color="2" fill="1" visible="no" active="no"/>
+<layer number="19" name="Unrouted" color="6" fill="1" visible="no" active="no"/>
+<layer number="20" name="Dimension" color="15" fill="1" visible="no" active="no"/>
+<layer number="21" name="tPlace" color="7" fill="1" visible="no" active="no"/>
+<layer number="22" name="bPlace" color="7" fill="1" visible="no" active="no"/>
+<layer number="23" name="tOrigins" color="15" fill="1" visible="no" active="no"/>
+<layer number="24" name="bOrigins" color="15" fill="1" visible="no" active="no"/>
+<layer number="25" name="tNames" color="7" fill="1" visible="no" active="no"/>
+<layer number="26" name="bNames" color="7" fill="1" visible="no" active="no"/>
+<layer number="27" name="tValues" color="7" fill="1" visible="no" active="no"/>
+<layer number="28" name="bValues" color="7" fill="1" visible="no" active="no"/>
 <layer number="29" name="tStop" color="7" fill="3" visible="no" active="no"/>
 <layer number="30" name="bStop" color="7" fill="6" visible="no" active="no"/>
@@
 <layer number="35" name="tGlue" color="7" fill="4" visible="no" active="no"/>
 <layer number="36" name="bGlue" color="7" fill="5" visible="no" active="no"/>
-<layer number="37" name="tTest" color="7" fill="1" visible="yes" active="no"/>
-<layer number="38" name="bTest" color="7" fill="1" visible="yes" active="no"/>
+<layer number="37" name="tTest" color="7" fill="1" visible="no" active="no"/>
+<layer number="38" name="bTest" color="7" fill="1" visible="no" active="no"/>
 <layer number="39" name="tKeepout" color="4" fill="11" visible="no" active="no"/>
 <layer number="40" name="bKeepout" color="1" fill="11" visible="no" active="no"/>
@@
 <layer number="44" name="Drills" color="7" fill="1" visible="no" active="no"/>
 <layer number="45" name="Holes" color="7" fill="1" visible="no" active="no"/>
-<layer number="46" name="Milling" color="3" fill="1" visible="yes" active="no"/>
-<layer number="47" name="Measures" color="7" fill="1" visible="yes" active="no"/>
-<layer number="48" name="Document" color="7" fill="1" visible="yes" active="no"/>
-<layer number="49" name="Reference" color="7" fill="1" visible="yes" active="no"/>
-<layer number="50" name="dxf" color="7" fill="1" visible="yes" active="no"/>
-<layer number="51" name="tDocu" color="7" fill="1" visible="yes" active="no"/>
-<layer number="52" name="bDocu" color="7" fill="1" visible="yes" active="no"/>
-<layer number="53" name="tGND_GNDA" color="7" fill="9" visible="yes" active="no"/>
-<layer number="54" name="bGND_GNDA" color="1" fill="9" visible="yes" active="no"/>
-<layer number="56" name="wert" color="7" fill="1" visible="yes" active="no"/>
+<layer number="46" name="Milling" color="3" fill="1" visible="no" active="no"/>
+<layer number="47" name="Measures" color="7" fill="1" visible="no" active="no"/>
+<layer number="48" name="Document" color="7" fill="1" visible="no" active="no"/>
+<layer number="49" name="Reference" color="7" fill="1" visible="no" active="no"/>
+<layer number="50" name="dxf" color="7" fill="1" visible="no" active="no"/>
+<layer number="51" name="tDocu" color="7" fill="1" visible="no" active="no"/>
+<layer number="52" name="bDocu" color="7" fill="1" visible="no" active="no"/>
+<layer number="53" name="tGND_GNDA" color="7" fill="9" visible="no" active="no"/>
+<layer number="54" name="bGND_GNDA" color="1" fill="9" visible="no" active="no"/>
+<layer number="56" name="wert" color="7" fill="1" visible="no" active="no"/>
 <layer number="90" name="Modules" color="5" fill="1" visible="yes" active="yes"/>
 <layer number="91" name="Nets" color="2" fill="1" visible="yes" active="yes"/>
@@
 <text x="198.12" y="129.54" size="1.778" layer="97">MCU</text>
 <text x="233.68" y="-93.98" size="1.778" layer="97">Diagnostic connector</text>
-<text x="10.16" y="-88.9" size="1.778" layer="97">qNode8-1.0.0+20160811</text>
+<text x="10.16" y="-88.9" size="1.778" layer="97">qNode8-1.0.1+20160812</text>
 <text x="10.16" y="-91.44" size="1.778" layer="97">(c) qyx@krtko.org, CC-BY-SA</text>
 <wire x1="10.16" y1="7.62" x2="332.74" y2="7.62" width="0.1524" layer="97"/>
@@
 <instance part="R8" gate="G$1" x="195.58" y="-121.92"/>
 <instance part="L2" gate="G$1" x="48.26" y="43.18" rot="R90"/>
-<instance part="C20" gate="G$1" x="38.1" y="35.56"/>
+<instance part="C20" gate="G$1" x="38.1" y="30.48"/>
 <instance part="GND34" gate="1" x="38.1" y="20.32"/>
 <instance part="BAT" gate="-1" x="27.94" y="111.76" rot="R180"/>
@@
 <pinref part="C20" gate="G$1" pin="2"/>
 <pinref part="GND34" gate="1" pin="GND"/>
-<wire x1="38.1" y1="30.48" x2="38.1" y2="22.86" width="0.1524" layer="91"/>
+<wire x1="38.1" y1="25.4" x2="38.1" y2="22.86" width="0.1524" layer="91"/>
 </segment>
 </net>
@@
 <wire x1="55.88" y1="43.18" x2="58.42" y2="43.18" width="0.1524" layer="91"/>
 <junction x="58.42" y="43.18"/>
+<wire x1="58.42" y1="43.18" x2="58.42" y2="48.26" width="0.1524" layer="91"/>
+<wire x1="58.42" y1="48.26" x2="60.96" y2="48.26" width="0.1524" layer="91"/>
+<label x="60.96" y="48.26" size="1.27" layer="95" xref="yes"/>
+</segment>
+<segment>
+<pinref part="IC1" gate="G$1" pin="PA9"/>
+<wire x1="302.26" y1="83.82" x2="307.34" y2="83.82" width="0.1524" layer="91"/>
+<label x="307.34" y="83.82" size="1.27" layer="95" xref="yes"/>
 </segment>
 </net>
@@
 </segment>
 </net>
-<net name="N$24" class="0">
+<net name="USB_VBUS" class="0">
 <segment>
 <pinref part="USB" gate="G$1" pin="VBUS"/>
 <pinref part="C20" gate="G$1" pin="1"/>
 <wire x1="25.4" y1="43.18" x2="38.1" y2="43.18" width="0.1524" layer="91"/>
-<wire x1="38.1" y1="43.18" x2="38.1" y2="38.1" width="0.1524" layer="91"/>
 <pinref part="L2" gate="G$1" pin="1"/>
+<wire x1="38.1" y1="43.18" x2="38.1" y2="33.02" width="0.1524" layer="91"/>
 <wire x1="38.1" y1="43.18" x2="40.64" y2="43.18" width="0.1524" layer="91"/>
 <junction x="38.1" y="43.18"/>
